Commit message: first commit

File: mir_description/urdf/include/mir_100.gazebo.xacro (robot description, xacro)
@@ -56,67 +56,3 @@
     </gazebo>
   </xacro:macro>
-  <xacro:macro name="camera" params="prefix">
-<joint name="camera_sensor_joint" type="fixed">
-            <axis xyz="0 1 0" />
-            <origin xyz="0 0 0 " rpy="0 0 0"/>
-            <parent link="${prefix}base_footprint"/>
-            <child link="camera_link"/>
-        </joint>
-        <link name="camera_link">
-            <collision>
-                <origin xyz="0 0 0" rpy="0 0 0"/>
-                <geometry>
-                    <box size="0.02 0.08 0.05"/>
-                </geometry>
-            </collision>
-            <visual>
-                <origin xyz="0 0 0" rpy="0 0 0"/>
-                <geometry>
-                    <box size="0.02 0.08 0.05"/>
-                </geometry>
-                <material name="iRobot/Green"/>
-            </visual>
-            <inertial>
-                <mass value="0.0001" />
-                <origin xyz="0 0 0" rpy="0 0 0"/>
-                <inertia ixx="0.0000001" ixy="0" ixz="0" iyy="0.0000001" iyz="0" izz="0.0000001" />
-            </inertial>
-        </link>
-        <gazebo reference="camera_link">
-            <sensor type="camera" name="camera">
-                <update_rate>30.0</update_rate>
-                <camera name="head">
-                    <horizontal_fov>1.3962634</horizontal_fov>
-                    <image>
-                        <width>800</width>
-                        <height>600</height>
-                        <format>R8G8B8</format>
-                    </image>
-                    <clip>
-                        <near>0.02</near>
-                        <far>300</far>
-                    </clip>
-                    <noise>
-                        <type>gaussian</type>
-                        <mean>0.0</mean>
-                        <stddev>0.007</stddev>
-                    </noise>
-                </camera>
-                <plugin name="camera_controller" filename="libgazebo_ros_camera.so">
-                    <alwaysOn>true</alwaysOn>
-                    <updateRate>0.0</updateRate>
-                    <cameraName>iRobot/camera</cameraName>
-                    <imageTopicName>image_raw</imageTopicName>
-                    <cameraInfoTopicName>camera_info</cameraInfoTopicName>
-                    <frameName>camera_link</frameName>
-                    <hackBaseline>0.07</hackBaseline>
-                    <distortionK1>0.0</distortionK1>
-                    <distortionK2>0.0</distortionK2>
-                    <distortionK3>0.0</distortionK3>
-                    <distortionT1>0.0</distortionT1>
-                    <distortionT2>0.0</distortionT2>
-                </plugin>
-            </sensor>
-    </gazebo>
-  </xacro:macro>
 </robot>

File: mir_description/urdf/include/mir_100_v1.urdf.xacro (robot description, xacro)
@@ -6,4 +6,5 @@
   <xacro:include filename="$(find mir_description)/urdf/include/mir_100.transmission.xacro" />
   <xacro:include filename="$(find mir_description)/urdf/include/sick_s300.urdf.xacro" />
+<xacro:include filename="$(find mir_description)/urdf/include/camera_sensor.urdf.xacro" />
   <xacro:property name="deg_to_rad" value="0.017453293" />
   <xacro:property name="mir_100_base_mass" value="58.0" />
@@ -179,4 +180,9 @@
     </joint>
     <xacro:sick_s300 prefix="${prefix}" link="back_laser_link" topic="b_scan" />
+<!-- start defining camera -->
+     <xacro:camera_sensor  xyz="0 0 1"
+                  rpy="0 0 0"
+                  parent="base_footprint" prefix="${prefix}" />
+<!-- end defining camera -->
     <!-- Ultrasound sensors -->
     <joint name="${prefix}us_1_joint" type="fixed">   <!-- right ultrasound -->
@@ -211,3 +217,9 @@
     <xacro:p3d_base_controller prefix="${prefix}" />
   </xacro:macro>
+<!-- start defining camera mir::
+     <xacro:camera_sensor xyz="0 0 ${0.04 + 0.02 + 0.04}"
+                  rpy="0 0 0"
+                  parent="mir::base_footprint">
+    </xacro:camera_sensor>
+end defining camera -->
 </robot>

File: mir_description/urdf/mir.urdf.xacro (robot description, xacro)
@@ -5,5 +5,4 @@
   <xacro:include filename="$(find mir_description)/urdf/include/mir_100_v1.urdf.xacro" />
   <xacro:include filename="$(find mir_description)/urdf/include/common.gazebo.xacro" />
-<!-- newly added-->
   <xacro:arg name="tf_prefix" default="" />
   <xacro:property name="tf_prefix_" value="$(arg tf_prefix)" />
@@ -14,6 +13,6 @@
     <xacro:property name="prefix" value="${tf_prefix_}/" />
   </xacro:unless>
-  <xacro:mir_100 prefix="${prefix}"/>
-  <xacro:controller_plugin_gazebo robot_namespace=""/>
+ <xacro:mir_100 prefix="${prefix}"/>
+ <xacro:controller_plugin_gazebo robot_namespace=""/>
   <!-- instead of the controller_plugin_gazebo, you can use the diffdrive controller like this:
     <xacro:diff_controller_plugin_gazebo prefix=""
